Commit message: Fixed the plugins in the urdf, added nav2 stack successfully (needs tuning)

File: urdf/youbot.urdf (robot description, URDF)
Before this commit: robot youbot, 22 links, 21 joints
Links:
- removed link base_laser_front_link
- added link base_laser_link, mass 0.1; collision box size=0.05 0.05 0.05; visual box size=0.05 0.05 0.05
- added link camera_link; visual box size=0.01 0.03 0.03
- added link camera_link_optical
Joints:
- removed joint base_laser_front_hokuyo_urg04_laser_joint
- added joint base_laser_joint: type fixed, parent base_link, child base_laser_link, origin xyz=0.3 0 0.03 rpy=0 0 0
- added joint camera_joint: type fixed, parent base_link, child camera_link, origin xyz=0.3 0 0.08 rpy=0 0 0
- added joint camera_optical_joint: type fixed, parent camera_link, child camera_link_optical, origin xyz=0.0 0.0 0.0 rpy=-1.570796 0 -1.570796
